File: kicad/esp32-c3/accra_A.kicad_sch (KiCad schematic)
At the start: 25 parts, among them IC1 ESP32-C3-WROOM-02-H4, J1 Conn_01x04_Male, J2 Conn_01x04_Male, J5 Conn_01x04, SW1 ALPS SKHH, U1 R-78C3.3-1.0, U2 SN65HVD232

Commit message: Changes power caps to SMD
Parts:
- C1, C2: footprint Capacitor_THT:CP_Radial_D6.3mm_P2.50mm -> Capacitor_SMD:C_0805_2012Metric_Pad1.18x1.45mm_HandSolder
Other:
- title: Accra version 2 -> Accra version 32C3
- moved on the sheet: D3, R2
Changed lines of the file:
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@@
   (paper "A4")
   (title_block
-    (title "Accra version 2")
+    (title "Accra version 32C3")
     (date "2022-06-09")
-    (rev "A")
+    (rev "B")
     (company "Grodans Paradis AB")
+    (comment 1 "VSCP A/D module with CAN/EWifi and BLE communication")
+    (comment 2 "https://www.vscp.org")
   )
   (junction (at 118.11 85.09) (diameter 0) (color 0 0 0 0)
@@
     (stroke (width 0) (type default) (color 0 0 0 0))
   )
-  (wire (pts (xy 223.52 143.51) (xy 223.52 144.78))
+  (wire (pts (xy 226.06 128.27) (xy 226.06 129.54))
     (stroke (width 0) (type default) (color 0 0 0 0))
   )
@@
     (stroke (width 0) (type default) (color 0 0 0 0))
   )
-  (wire (pts (xy 223.52 152.4) (xy 223.52 156.21))
+  (wire (pts (xy 226.06 137.16) (xy 226.06 140.97))
     (stroke (width 0) (type default) (color 0 0 0 0))
   )
@@
     (stroke (width 0) (type default) (color 0 0 0 0))
   )
-  (wire (pts (xy 214.63 130.81) (xy 223.52 130.81))
+  (wire (pts (xy 217.17 115.57) (xy 226.06 115.57))
     (stroke (width 0) (type default) (color 0 0 0 0))
   )
@@
     (stroke (width 0) (type default) (color 0 0 0 0))
   )
-  (wire (pts (xy 223.52 130.81) (xy 223.52 135.89))
+  (wire (pts (xy 226.06 115.57) (xy 226.06 120.65))
     (stroke (width 0) (type default) (color 0 0 0 0))
   )
@@
     (effects (font (size 1.27 1.27)) (justify left bottom))
   )
-  (label "status" (at 214.63 130.81 0)
+  (label "status" (at 217.17 115.57 0)
     (effects (font (size 1.27 1.27)) (justify left bottom))
   )
@@
     )
   )
-  (symbol (lib_id "Device:R") (at 223.52 139.7 0) (unit 1)
-    (in_bom yes) (on_board yes) (fields_autoplaced)
-    (property "Reference" "R2" (id 0) (at 225.298 138.8653 0)
-      (effects (font (size 1.27 1.27)) (justify left))
-    )
-    (property "Value" "10K" (id 1) (at 225.298 141.4022 0)
-      (effects (font (size 1.27 1.27)) (justify left))
-    )
-    (property "Footprint" "Resistor_SMD:R_0805_2012Metric" (id 2) (at 221.742 139.7 90)
-      (effects (font (size 1.27 1.27)) hide)
-    )
-    (property "Datasheet" "~" (id 3) (at 223.52 139.7 0)
-      (effects (font (size 1.27 1.27)) hide)
-    )
-    (pin "1")
-    (pin "2")
-  )
-  (symbol (lib_id "Device:LED") (at 223.52 148.59 90) (unit 1)
-    (in_bom yes) (on_board yes) (fields_autoplaced)
-    (property "Reference" "D3" (id 0) (at 226.441 149.3428 90)
+  (symbol (lib_id "Device:R") (at 226.06 124.46 0) (unit 1)
+    (in_bom yes) (on_board yes) (fields_autoplaced)
+    (property "Reference" "R2" (id 0) (at 227.838 123.6253 0)
+      (effects (font (size 1.27 1.27)) (justify left))
+    )
+    (property "Value" "10K" (id 1) (at 227.838 126.1622 0)
+      (effects (font (size 1.27 1.27)) (justify left))
+    )
+    (property "Footprint" "Resistor_SMD:R_0805_2012Metric" (id 2) (at 224.282 124.46 90)
+      (effects (font (size 1.27 1.27)) hide)
+    )
+    (property "Datasheet" "~" (id 3) (at 226.06 124.46 0)
+      (effects (font (size 1.27 1.27)) hide)
+    )
+    (pin "1")
+    (pin "2")
+  )
+  (symbol (lib_id "Device:LED") (at 226.06 133.35 90) (unit 1)
+    (in_bom yes) (on_board yes) (fields_autoplaced)
+    (property "Reference" "D3" (id 0) (at 228.981 134.1028 90)
       (effects (font (size 1.27 1.27)) (justify right))
     )
-    (property "Value" "Status" (id 1) (at 226.441 151.8797 90)
+    (property "Value" "Status" (id 1) (at 228.981 136.6397 90)
       (effects (font (size 1.27 1.27)) (justify right))
     )
-    (property "Footprint" "LED_SMD:LED_0805_2012Metric" (id 2) (at 223.52 148.59 0)
-      (effects (font (size 1.27 1.27)) hide)
-    )
-    (property "Datasheet" "~" (id 3) (at 223.52 148.59 0)
+    (property "Footprint" "LED_SMD:LED_0805_2012Metric" (id 2) (at 226.06 133.35 0)
+      (effects (font (size 1.27 1.27)) hide)
+    )
+    (property "Datasheet" "~" (id 3) (at 226.06 133.35 0)
       (effects (font (size 1.27 1.27)) hide)
     )
@@
     (pin "1")
   )
-  (symbol (lib_id "power:GND") (at 223.52 156.21 0) (unit 1)
-    (in_bom yes) (on_board yes) (fields_autoplaced)
-    (property "Reference" "#PWR0124" (id 0) (at 223.52 162.56 0)
-      (effects (font (size 1.27 1.27)) hide)
-    )
-    (property "Value" "GND" (id 1) (at 223.52 160.6534 0))
-    (property "Footprint" "" (id 2) (at 223.52 156.21 0)
-      (effects (font (size 1.27 1.27)) hide)
-    )
-    (property "Datasheet" "" (id 3) (at 223.52 156.21 0)
+  (symbol (lib_id "power:GND") (at 226.06 140.97 0) (unit 1)
+    (in_bom yes) (on_board yes) (fields_autoplaced)
+    (property "Reference" "#PWR0124" (id 0) (at 226.06 147.32 0)
+      (effects (font (size 1.27 1.27)) hide)
+    )
+    (property "Value" "GND" (id 1) (at 226.06 145.4134 0))
+    (property "Footprint" "" (id 2) (at 226.06 140.97 0)
+      (effects (font (size 1.27 1.27)) hide)
+    )
+    (property "Datasheet" "" (id 3) (at 226.06 140.97 0)
       (effects (font (size 1.27 1.27)) hide)
     )
@@
       (effects (font (size 1.27 1.27)) (justify left))
     )
-    (property "Footprint" "Capacitor_THT:CP_Radial_D6.3mm_P2.50mm" (id 2) (at 71.12 172.72 0)
+    (property "Footprint" "Capacitor_SMD:C_0805_2012Metric_Pad1.18x1.45mm_HandSolder" (id 2) (at 71.12 172.72 0)
       (effects (font (size 1.27 1.27)) hide)
     )
@@
       (effects (font (size 1.27 1.27)) (justify left))
     )
-    (property "Footprint" "Capacitor_THT:CP_Radial_D6.3mm_P2.50mm" (id 2) (at 35.56 172.72 0)
+    (property "Footprint" "Capacitor_SMD:C_0805_2012Metric_Pad1.18x1.45mm_HandSolder" (id 2) (at 35.56 172.72 0)
       (effects (font (size 1.27 1.27)) hide)
     )
@@
     )
     (path "/e9ba72cc-4567-4018-b654-0ead0f54c894"
-      (reference "C1") (unit 1) (value "22uF") (footprint "Capacitor_THT:CP_Radial_D6.3mm_P2.50mm")
+      (reference "C1") (unit 1) (value "22uF") (footprint "Capacitor_SMD:C_0805_2012Metric_Pad1.18x1.45mm_HandSolder")
     )
     (path "/54bd990f-4542-47f8-98cd-a4208c34c341"
-      (reference "C2") (unit 1) (value "10uF") (footprint "Capacitor_THT:CP_Radial_D6.3mm_P2.50mm")
+      (reference "C2") (unit 1) (value "10uF") (footprint "Capacitor_SMD:C_0805_2012Metric_Pad1.18x1.45mm_HandSolder")
     )
     (path "/3c1cde26-c75a-497a-aacd-b921320388d7"

Commit message: Added protection diod on input
Parts:
- added D4: 1N5819, Diode_SMD:D_SOD-123, symbol Diode:1N5819
- added J6, J7: Conn_01x04, Connector_Molex:Molex_KK-254_AE-6410-04A_1x04_P2.54mm_Vertical, symbol Connector_Generic:Conn_01x04
Connections:
- net +28V: now also J6.1 (Pin_1), J7.1 (Pin_1)
- net +3V3: now also D4.1 (K); no longer C2.1, U1.3 (OUT)
- net GND: now also J6.4 (Pin_4), J7.4 (Pin_4)
- net CANL: now reaches D1.1 (K), J1.2 (Pin_2), JP1.1 (A), U2.6 (CANL)
- net CANL: now also J6.3 (Pin_3), J7.3 (Pin_3)
- net CANH: now reaches D1.2 (K), J1.3 (Pin_3), R17.2, U2.7 (CANH)
- net CANH: now also J6.2 (Pin_2), J7.2 (Pin_2)
- new net: C2.1, D4.2 (A), U1.3 (OUT)
